File: vigoleno.kicad_pcb (KiCad board)
At the start: 6 copper layers, 181 parts, among them J1 9P-MSD-PP-V2, J3 USB_OTG, J4 IPEX RF Coaxial Connector SMD, M1 MODULE_RTL8188, U1 MT29F8G08ABABA, U2 ISL8022, U3 ALLWINNER-A13(176-LQFP), U4 TLV62569-SOT23-6, U5 TPS62233DRYR, U6 AS4C256M16D3A-12BAN(96-FBGA)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

Commit message: update Dec 20 2018
Routing:
- net /DDR3-ODT: track 63.6 -> 28.1 mm
- net /A5: track 60.1 -> 25.2 mm
- net /A2: track 44.5 -> 13.0 mm, vias 2 -> 1
- net /A3: track 43.2 -> 13.1 mm
- net /DDR3-RST: track 48.7 -> 19.1 mm
- net /A7: track 51.3 -> 23.4 mm
- net /A0: track 41.6 -> 14.5 mm
- net /BA0: track 42.2 -> 16.2 mm
- net /BA2: track 40.5 -> 16.7 mm
- net /WE: track 39.7 -> 16.7 mm
- net /CAS: track 39.2 -> 17.1 mm
- net /RAS: track 39.0 -> 17.7 mm
- net /A9: track 0.00 -> 19.2 mm, vias 0 -> 2
- net /A13: track 0.00 -> 14.7 mm, vias 0 -> 2
- net /A14: track 32.2 -> 21.2 mm
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