File: vigoleno.kicad_pcb (KiCad board)
At the start: 6 copper layers, 181 parts, among them J1 9P-MSD-PP-V2, J3 USB_OTG, J4 IPEX RF Coaxial Connector SMD, M1 MODULE_RTL8188, U1 MT29F8G08ABABA, U2 ISL8022, U3 ALLWINNER-A13(176-LQFP), U4 TLV62569-SOT23-6, U5 TPS62233DRYR, U6 AS4C256M16D3A-12BAN(96-FBGA), U7 MCP130T-300ITT, Y1 Crystal_GND24_24MHz

Commit message: update Dec 21 2018
Parts:
- moved U1 22.0 mm to (578.1, -475.9)
Routing:
- net /A3: track 13.1 -> 43.1 mm
- net /A2: track 13.0 -> 43.0 mm, vias 1 -> 2
- net /A9: track 19.2 -> 47.3 mm
- net /DDR3-RST: track 19.1 -> 47.1 mm
- net /A13: track 14.7 -> 42.4 mm, vias 2 -> 3
- net /A0: track 14.5 -> 41.4 mm
- net /BA0: track 16.2 -> 42.2 mm
- net /A7: track 23.4 -> 49.3 mm
- net /DDR3-ODT: track 28.1 -> 53.9 mm
- net /BA2: track 16.7 -> 40.5 mm
- net /A5: track 25.2 -> 48.7 mm
- net /WE: track 16.7 -> 40.1 mm
- net /CAS: track 17.1 -> 39.2 mm
- net /RAS: track 17.7 -> 38.9 mm
- net /D4: track 28.0 -> 37.0 mm
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
Commit message: update Dec 24 2018
Routing:
- net /A13: track 42.4 -> 59.8 mm
- net /A2: track 43.0 -> 27.2 mm
- net /WE: track 40.1 -> 55.8 mm
- net /DDR3-RST: track 47.1 -> 58.0 mm
- net /A9: track 47.3 -> 58.1 mm
- net /A5: track 48.7 -> 58.0 mm
- net /A7: track 49.3 -> 58.1 mm
- net /CK: track 24.1 -> 19.5 mm
- net /DDR3-ODT: track 53.9 -> 58.0 mm
- net /BA1: track 27.8 -> 24.2 mm
- net /A12: track 27.4 -> 24.0 mm
- net /A3: track 43.1 -> 46.5 mm
- net /A0: track 41.4 -> 44.7 mm
- net /BA0: track 42.2 -> 45.3 mm
- net /BA2: track 40.5 -> 43.6 mm
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
Commit message: update Dec 25 2018
Routing:
- net /A10: track 22.4 -> 58.0 mm
- net /A12: track 24.0 -> 58.0 mm
- net /BA1: track 24.2 -> 58.0 mm
- net /A4: track 24.5 -> 58.1 mm
- net /A1: track 26.7 -> 58.1 mm
- net /A6: track 27.0 -> 58.1 mm
- net /A2: track 27.2 -> 58.0 mm
- net /A11: track 29.4 -> 58.0 mm
- net /A8: track 30.1 -> 58.1 mm
- net /A14: track 30.6 -> 58.0 mm
- net /CAS: track 41.9 -> 67.7 mm
- net /D10: track 14.5 -> 38.0 mm
- net /D12: track 15.4 -> 38.0 mm
- net /DQS1-N: track 16.2 -> 38.0 mm
- net /D3: track 16.3 -> 38.0 mm
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
Commit message: update JAN 5 2019
Parts:
- moved C80 162.0 mm to (691.1, -460.0)
- moved R19 162.0 mm to (693.3, -451.9)
- moved C73 162.0 mm to (701.8, -458.9)
- moved J1 162.0 mm to (703.9, -470.8)
- moved L5 162.0 mm to (695.5, -457.0)
- moved R23 162.0 mm to (706.4, -455.5)
- moved RN15 162.0 mm to (700.5, -452.3)
- moved M1 101.0 mm to (645.2, -426.0)
- moved U1 23.3 mm to (574.8, -452.9), turned to 90 degrees
Routing:
- net /D14: track 15.2 -> 55.0 mm
- net /D8: track 21.7 -> 55.1 mm
- net /DQS0: track 38.1 -> 61.5 mm
- net /DQS0-N: track 38.0 -> 61.3 mm
- net /DM0: track 38.0 -> 61.2 mm
- net /DQS1: track 38.0 -> 61.1 mm
- net /CKE: track 37.0 -> 55.1 mm
- net /D9: track 38.0 -> 55.1 mm
- net /D6: track 38.0 -> 55.0 mm
- net /D1: track 38.0 -> 55.0 mm
- net /DM1: track 38.0 -> 55.0 mm
- net /D10: track 38.0 -> 55.0 mm
- net /D3: track 38.0 -> 55.0 mm
- net /D5: track 38.0 -> 55.0 mm
- net /DQS1-N: track 38.0 -> 55.0 mm
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
Commit message: update Jan 6 2019
Parts:
- C73, C80, J1, L5, R19, R23, RN15, U1: moved to F.Cu
- J3: footprint MyKiCadLib:USB_Micro_B_Female_SMD -> MyKiCadLib:USB_Micro_3MV2
- moved MENU1 403.8 mm to (578.1, -403.3)
- moved VOL+1 403.6 mm to (591.9, -403.3)
- moved ENTER1 398.5 mm to (571.2, -403.3)
- moved RN1 398.0 mm to (601.0, -414.9)
- moved VOL-1 378.1 mm to (585.0, -403.3)
- moved HOME1 375.3 mm to (564.3, -403.3)
- moved L6 360.4 mm to (609.2, -495.1)
- moved C97 352.6 mm to (621.1, -499.4)
- moved C23 351.4 mm to (581.0, -447.9), turned to 90 degrees
- moved C16 350.6 mm to (555.3, -447.8), turned to 90 degrees
- moved C26 350.6 mm to (582.0, -447.9), turned to 90 degrees
- moved C82 349.8 mm to (560.6, -433.7)
- moved RN2 348.6 mm to (554.4, -451.9), turned to 180 degrees
- moved C14 346.6 mm to (554.1, -447.8), turned to 90 degrees
- moved H-P1 346.6 mm to (602.5, -405.3)
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Connections:
- J1 pad 10: Net-(J1-Pad10) -> GND
- R16 pad 2: Net-(R16-Pad2) -> /+3.0VA
- R23 pad 2: Net-(J1-Pad10) -> /SD0CARD-DETECT
- RN15 pad 1: /SDC0-DATA2 -> /SD0CARD-DETECT
- RN15 pad 2: /SDC0-DATA0 -> /SDC0-DATA1
- RN15 pad 3: /SDC0-DATA1 -> /SDC0-DATA0
- RN15 pad 4: /SD0CARD-DETECT -> /SDC0-DATA2

Commit message: update Jan 7 2019
Parts:
- C1, C2, C36, C37, C55, C56, C58, C59, C62, C69, C97, C98, D1, J1, J4, JP2, L1, L2, L3, L4, L6, ON1, R10, R11, R12, R24, R5, R6, R7, R8, TP0, TP1, TP2, TP3, TP4, U2, U4, U5: moved to B.Cu
- moved TP0 507.9 mm to (619.0, -410.4)
- moved C68 498.2 mm to (627.2, -410.6), turned to 90 degrees
- moved C65 496.6 mm to (625.9, -410.6), turned to 90 degrees
- moved C61 492.9 mm to (624.5, -410.6), turned to 90 degrees
- moved C71 488.9 mm to (630.0, -410.6), turned to 90 degrees
- moved C70 485.1 mm to (628.6, -410.6), turned to 90 degrees
- moved ON1 477.4 mm to (626.4, -410.5)
- moved R24 476.0 mm to (629.0, -410.5)
- moved U5 473.7 mm to (615.0, -412.9), turned to 270 degrees
- moved C69 473.4 mm to (613.3, -412.6), turned to 90 degrees
- moved TP4 473.1 mm to (613.4, -418.0), turned to 270 degrees
- moved C62 469.5 mm to (616.9, -412.8), turned to 90 degrees
- moved L4 469.3 mm to (614.5, -415.4), turned to 180 degrees
- moved R11 440.3 mm to (607.4, -414.6), turned to 270 degrees
- moved U4 439.8 mm to (610.3, -416.2), turned to 270 degrees
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Routing:
- net /PIN12_NWE: track 0.00 -> 43.0 mm
- net /PIN13_NALE: track 0.00 -> 42.0 mm
- net /PIN14_NCLE: track 0.00 -> 41.8 mm
- net /PIN18_NRB0: track 0.00 -> 40.2 mm
- net /PIN17_NRE: track 0.00 -> 39.4 mm
- net /SVREF: track 0.00 -> 11.8 mm
- net /TPY1: track 0.00 -> 10.7 mm
- net Net-(C32-Pad1): track 0.00 -> 9.17 mm
- net Net-(C31-Pad1): track 0.00 -> 9.01 mm
- net /TPX1: track 0.00 -> 8.80 mm
- net GND: track 43.2 -> 51.7 mm, vias 2 -> 6
- net +3V3: track 0.00 -> 7.84 mm
- net Net-(JP1-Pad2): track 0.00 -> 7.71 mm
- net Net-(C43-Pad1): track 0.00 -> 7.00 mm
- net /TPY2: track 0.00 -> 5.96 mm
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Other:
- board outline added: 80.8 x 53.2 mm
