File: vigoleno.sch (KiCad schematic (older format))
At the start: 181 parts, among them J1 9P-MSD-PP-V2, J3 USB_OTG, J4 IPEX RF Coaxial Connector SMD, M1 MODULE_RTL8188, U1 MT29F8G08ABABA, U2 ISL8022, U3 ALLWINNER-A13(176-LQFP), U4 TLV62569-SOT23-6, U5 TPS62233DRYR, U6 AS4C256M16D3A-12BAN(96-FBGA)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

Commit message: update Jan 6 2019
Parts:
- J3: footprint MyKiCadLib:USB_Micro_B_Female_SMD -> MyKiCadLib:USB_Micro_3MV2
Connections:
- net +3.0VA: now also R16.2
- net GND: now also J1.10 (GND)
- net SD0CARD-DETECT: now also R23.2, RN15.1 (R1.1); no longer RN15.4 (R4.1)
- net SDC0-DATA0: now also RN15.3 (R3.1); no longer RN15.2 (R2.1)
- net SDC0-DATA1: now also RN15.2 (R2.1); no longer RN15.3 (R3.1)
- net SDC0-DATA2: now also RN15.4 (R4.1); no longer RN15.1 (R1.1)
Other:
- moved on the sheet: R23
Changed lines of the file:
@@
 Connection ~ 15700 11900
 Connection ~ 15700 12200
-Wire Wire Line
-	15500 12300 16150 12300
 $Comp
 L Device:R R23
 U 1 1 5C07273D
-P 15800 12400
-F 0 "R23" V 15750 12200 50  0000 C CNN
-F 1 "R0402/10K" V 15750 12750 50  0000 C CNN
-F 2 "MyKiCadLib:R0402_HandSoldering" V 15730 12400 50  0001 C CNN
-F 3 "~" H 15800 12400 50  0001 C CNN
-	1    15800 12400
+P 16350 12300
+F 0 "R23" V 16400 12500 50  0000 C CNN
+F 1 "R0402/10K" V 16400 11900 50  0000 C CNN
+F 2 "MyKiCadLib:R0402_HandSoldering" V 16280 12300 50  0001 C CNN
+F 3 "~" H 16350 12300 50  0001 C CNN
+	1    16350 12300
 	0    1    1    0
 $EndComp
 Wire Wire Line
-	15650 12400 15500 12400
-Wire Wire Line
-	15950 12400 16650 12400
-Wire Wire Line
-	16650 12400 16650 12200
+	16650 12400 16650 12300
 Wire Wire Line
 	15700 12200 16650 12200
@@
 	13600 12000 13600 11750
 Wire Wire Line
-	14250 12400 13750 12400
-Wire Wire Line
-	13750 12400 13750 11800
-Wire Wire Line
 	13600 12000 12900 12000
 Connection ~ 13600 12000
 Wire Wire Line
 	14250 12100 12900 12100
-Wire Wire Line
-	13750 12400 12900 12400
-Connection ~ 13750 12400
 Text Label 12900 11900 0    50   ~ 0
 SDC0-DATA3
@@
 Text Label 12550 8500 0    50   ~ 0
 LRADC
-$Comp
-L Mylib:+3.0VA #PWR031
-U 1 1 5D6AF1B8
-P 13150 8000
-F 0 "#PWR031" H 13150 7850 50  0001 C CNN
-F 1 "+3.0VA" H 13165 8173 50  0000 C CNN
-F 2 "" H 13150 8000 50  0001 C CNN
-F 3 "" H 13150 8000 50  0001 C CNN
-	1    13150 8000
-	1    0    0    -1
-$EndComp
-Wire Wire Line
-	13150 8000 13150 8100
 Text Label 4900 5600 0    50   ~ 0
 UBOOT
@@
 F 0 "J3" H 21355 3067 50  0000 C CNN
 F 1 "USB_OTG" H 21355 2976 50  0000 C CNN
-F 2 "MyKiCadLib:USB_Micro_B_Female_SMD" H 21450 2550 50  0001 C CNN
+F 2 "MyKiCadLib:USB_Micro_3MV2" H 21450 2550 50  0001 C CNN
 F 3 " ~" H 21450 2550 50  0001 C CNN
 	1    21300 2600
@@
 Wire Wire Line
 	12900 11900 14250 11900
-Wire Wire Line
-	14050 11800 14050 12500
-Wire Wire Line
-	14050 12500 12900 12500
 Text Label 12900 12500 0    50   ~ 0
 SD0CARD-DETECT
@@
 	12800 12400 12900 12500
 Wire Wire Line
-	12900 12300 13950 12300
-Wire Wire Line
-	12900 12200 13850 12200
-Wire Wire Line
-	13850 11800 13850 12200
-Connection ~ 13850 12200
-Wire Wire Line
-	13850 12200 14250 12200
-Wire Wire Line
-	13950 11800 13950 12300
-Connection ~ 13950 12300
-Wire Wire Line
-	13950 12300 14250 12300
+	12900 12300 13850 12300
 Text Label 21550 9900 2    50   ~ 0
 LCD-D18
@@
 Wire Wire Line
 	21550 11300 21550 11400
+Connection ~ 21550 11400
+Wire Wire Line
+	12900 12400 14050 12400
+Wire Wire Line
+	13750 11800 13750 12500
+Wire Wire Line
+	12900 12500 13750 12500
+Wire Wire Line
+	12900 12200 13950 12200
+Wire Wire Line
+	13850 11800 13850 12300
+Connection ~ 13850 12300
+Wire Wire Line
+	13850 12300 14250 12300
+Wire Wire Line
+	13950 11800 13950 12200
+Connection ~ 13950 12200
+Wire Wire Line
+	13950 12200 14250 12200
+Wire Wire Line
+	14050 11800 14050 12400
+Connection ~ 14050 12400
+Wire Wire Line
+	14050 12400 14250 12400
+Wire Wire Line
+	15500 12400 16650 12400
+Wire Wire Line
+	15500 12300 16200 12300
+Wire Wire Line
+	16500 12300 16650 12300
+Connection ~ 16650 12300
+Wire Wire Line
+	16650 12300 16650 12200
 Wire Wire Line
 	2350 11250 3600 11250
@@
 Wire Bus Line
 	10950 1250 10950 6250
-Connection ~ 21550 11400
+$Comp
+L Mylib:+3.0VA #PWR0101
+U 1 1 5CE85E3A
+P 13150 8000
+F 0 "#PWR0101" H 13150 7850 50  0001 C CNN
+F 1 "+3.0VA" H 13165 8173 50  0000 C CNN
+F 2 "" H 13150 8000 50  0001 C CNN
+F 3 "" H 13150 8000 50  0001 C CNN
+	1    13150 8000
+	1    0    0    -1
+$EndComp
+Wire Wire Line
+	13150 8000 13150 8100
+Text Label 13150 8050 0    50   ~ 0
++3.0VA
 $EndSCHEMATC
