File: PCB/vigoleno/vigoleno.kicad_pcb (KiCad board)
At the start: 6 copper layers, 80.8 x 53.2 mm, 181 parts, among them J1 9P-MSD-PP-V2, J3 USB_OTG, J4 IPEX RF Coaxial Connector SMD, M1 MODULE_RTL8188, U1 MT29F8G08ABABA, U2 ISL8022, U3 ALLWINNER-A13(176-LQFP), U4 TLV62569-SOT23-6, U5 TPS62233DRYR, U6 AS4C256M16D3A-12BAN(96-FBGA), U7 MCP130T-300ITT, Y1 Crystal_GND24_24MHz

Commit message: update Jan 8 2019
Parts:
- C1, C2, C36, C37, C55, C56, C58, C59, C62, C69, L1, L2, L3, L4, ON1, R10, R11, R12, R24, R5, R6, R7, R8, TP0, TP1, TP2, TP3, TP4, U2, U4, U5: moved to F.Cu
- C73, C80, L5, R19, R23, RN15: moved to B.Cu
- moved TP3 20.4 mm to (623.6, -410.7), turned to 90 degrees
- moved C59 18.7 mm to (624.9, -412.9), turned to 0 degrees
- moved J3 18.2 mm to (632.4, -410.8), turned to 90 degrees
- moved C71 16.9 mm to (616.6, -421.0), turned to 270 degrees
- moved TP1 15.4 mm to (610.6, -408.8)
- moved TP2 15.4 mm to (614.0, -408.8)
- moved L3 15.1 mm to (624.9, -415.8), turned to 270 degrees
- moved R12 15.0 mm to (621.8, -412.8), turned to 180 degrees
- moved C70 14.9 mm to (617.9, -421.0), turned to 270 degrees
- moved C56 13.9 mm to (620.0, -409.9), turned to 90 degrees
- moved C55 13.9 mm to (604.6, -409.9), turned to 90 degrees
- moved L2 13.5 mm to (616.5, -410.2), turned to 270 degrees
- moved L1 13.5 mm to (608.0, -410.2), turned to 270 degrees
- moved C37 13.2 mm to (618.8, -410.4), turned to 270 degrees
- moved C36 13.2 mm to (605.8, -410.4), turned to 270 degrees
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Connections:
- GPIO1 pad 27: /PIN28 -> /PIN28_NDQS
- RN2 pad 1: /PIN18_NRB0 -> /PIN16_NCE0
- RN2 pad 2: /PIN16_NCE0 -> /PIN18_NRB0
Routing:
- net GND: track 51.7 -> 151.3 mm
- net /UBOOT: track 0.00 -> 95.5 mm, vias 0 -> 2
- net Net-(H-P1-Pad4): track 2.25 -> 76.4 mm, vias 1 -> 4
- net /UDM1: track 0.00 -> 71.0 mm, vias 0 -> 2
- net /UDP1: track 0.00 -> 71.0 mm, vias 0 -> 2
- net Net-(H-P1-Pad11): track 2.04 -> 72.7 mm, vias 1 -> 2
- net Net-(H-P1-Pad10): track 2.75 -> 73.1 mm, vias 1 -> 2
- net /RESET-N: track 0.00 -> 62.6 mm, vias 0 -> 2
- net Net-(C4-Pad2): track 0.00 -> 49.8 mm, vias 0 -> 2
- net Net-(C40-Pad2): track 0.00 -> 48.4 mm, vias 0 -> 2
- net /PIN20_NDQ0: track 0.00 -> 45.1 mm, vias 0 -> 2
- net /PIN21_NDQ1: track 0.00 -> 45.0 mm, vias 0 -> 2
- net /PIN22_NDQ2: track 0.00 -> 43.6 mm, vias 0 -> 2
- net /PIN23_NDQ3: track 0.00 -> 42.4 mm, vias 0 -> 2
- net /PIN24_NDQ4: track 0.00 -> 39.3 mm, vias 0 -> 2
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Other:
- board size 80.8 x 53.2 mm -> 80.8 x 55 mm
- net class Default: clearance 0.15 -> 0.2
- rule trace_clearance: 0.15 -> 0.2

Commit message: update Feb 1
Parts:
- moved R23 16.9 mm to (613.5, -437.4), turned to 0 degrees
- moved RN15 14.8 mm to (613.4, -434.9), turned to 180 degrees
- moved R19 13.3 mm to (613.4, -432.5), turned to 180 degrees
- moved C80 9.94 mm to (612.3, -424.7), turned to 0 degrees
- moved C73 9.46 mm to (612.3, -426.1), turned to 0 degrees
- moved L5 9.40 mm to (612.3, -427.8), turned to 0 degrees
Routing:
- net Net-(C73-Pad2): track 0.00 -> 18.6 mm
- net /PIN4_TWI0-SCK: track 0.00 -> 14.9 mm
- net /SDC0-DATA2: track 0.00 -> 6.03 mm
- net /SD0CARD-DETECT: track 0.00 -> 5.96 mm
- net /SDC0-DATA1: track 0.00 -> 5.54 mm
- net /SDC0-DATA0: track 0.00 -> 5.46 mm
- net /SDC0-CMD: track 0.00 -> 3.89 mm, vias 0 -> 2
- net /LRADC: track 33.1 -> 34.0 mm

Commit message: update Feb 25 2019
Routing:
- net /+1.5V: track 0.00 -> 25.8 mm, vias 0 -> 5
- net /+1.2V-CPU: track 0.00 -> 24.4 mm, vias 0 -> 4
- net /+1.2V-INT: track 0.00 -> 20.3 mm, vias 0 -> 4
- net +3V3: track 15.5 -> 32.3 mm, vias 0 -> 3
- net Net-(C20-Pad1): track 0.00 -> 8.24 mm, vias 0 -> 1
- net /+3.0VA: track 0.00 -> 7.22 mm, vias 0 -> 1
- net /SVREF: track 11.8 -> 18.0 mm, vias 0 -> 1
- net Net-(C21-Pad1): track 0.00 -> 6.03 mm, vias 0 -> 1
- net Net-(R13-Pad2): track 0.00 -> 5.73 mm, vias 0 -> 1
- net Net-(C34-Pad1): track 0.00 -> 3.80 mm, vias 0 -> 1
- net Net-(H-P1-Pad4): track 76.4 -> 75.6 mm

Commit message: update Feb 27
Routing:
- net /UDP0: track 0.00 -> 49.9 mm, vias 0 -> 3
- net /UDM0: track 0.00 -> 49.8 mm, vias 0 -> 3
- net GND: track 151.3 -> 191.6 mm
- net /TPY2: track 5.96 -> 30.2 mm, vias 0 -> 1
- net /TPX2: track 5.70 -> 29.1 mm, vias 0 -> 1
- net /TPY1: track 10.7 -> 33.2 mm, vias 0 -> 1
- net /TPX1: track 8.80 -> 30.0 mm, vias 0 -> 1
- net /LCD-CLK: track 0.00 -> 9.11 mm, vias 0 -> 1
- net +3V3: track 32.3 -> 41.4 mm
- net /PIN35: track 0.00 -> 8.49 mm, vias 0 -> 1
- net /LCD-HSYNC: track 0.00 -> 8.39 mm, vias 0 -> 1
- net /LCD-DE: track 0.00 -> 8.20 mm, vias 0 -> 1
- net /PIN36: track 0.00 -> 7.72 mm, vias 0 -> 1
- net /PIN33: track 0.00 -> 7.14 mm, vias 0 -> 1
- net /LCD-VSYNC: track 0.00 -> 7.10 mm, vias 0 -> 1
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
Commit message: update March 52019
Parts:
- C61, C65, C68, C70, C71, D2, D3: moved to B.Cu
- DEBUG1: footprint Connector_PinHeader_2.54mm:PinHeader_1x03_P2.54mm_Horizontal -> Connector_Molex:Molex_CLIK-Mate_502585-0370_1x03-1MP_P1.50mm_Horizontal; moved to B.Cu
- moved DEBUG1 69.5 mm to (556.6, -452.7)
- moved D3 35.1 mm to (590.6, -442.2), turned to 180 degrees
- moved D2 35.1 mm to (590.6, -439.1), turned to 180 degrees
- moved C55 24.2 mm to (624.2, -424.1), turned to 270 degrees
- moved C73 23.5 mm to (614.3, -449.5)
- moved C80 23.5 mm to (614.3, -448.1)
- moved L5 23.5 mm to (614.3, -451.2)
- moved C36 21.6 mm to (623.0, -423.5), turned to 90 degrees
- moved R19 19.9 mm to (614.3, -452.4)
- moved RN15 19.9 mm to (614.3, -454.8)
- moved R23 19.9 mm to (614.3, -457.3)
- moved L1 18.6 mm to (620.8, -423.8), turned to 90 degrees
- moved C56 18.1 mm to (608.9, -424.1), turned to 270 degrees
- moved TP1 18.0 mm to (618.3, -425.1), turned to 180 degrees
- moved J1 17.7 mm to (623.4, -449.6)
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Connections:
- GPIO1 pad 5: /REST-N -> /RESET-N
Routing:
- net /PIN36: track 7.72 -> 39.2 mm, vias 1 -> 2
- net /TPX2: track 29.1 -> 59.8 mm, vias 1 -> 3
- net /PIN35: track 8.49 -> 37.9 mm, vias 1 -> 2
- net /TPY2: track 30.2 -> 58.3 mm, vias 1 -> 3
- net /UDP1: track 71.0 -> 97.9 mm, vias 2 -> 3
- net GND: track 191.6 -> 164.8 mm, vias 6 -> 5
- net /UDM1: track 71.0 -> 97.8 mm, vias 2 -> 3
- net /TPY1: track 33.2 -> 10.7 mm, vias 1 -> 0
- net /TPX1: track 30.0 -> 8.77 mm
- net /UBOOT: track 95.5 -> 74.6 mm
- net Net-(C73-Pad2): track 18.6 -> 0.00 mm
- net /LCD-VSYNC: track 7.10 -> 21.7 mm, vias 1 -> 2
- net /LCD-DE: track 8.20 -> 22.7 mm, vias 1 -> 2
- net /LCD-HSYNC: track 8.39 -> 20.2 mm, vias 1 -> 2
- net +3V3: track 41.4 -> 52.1 mm
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Other:
- board size 80.8 x 55 mm -> 80.8 x 50 mm
