File: PCB/vigoleno/vigoleno.sch (KiCad schematic (older format))
At the start: 181 parts, among them J1 9P-MSD-PP-V2, J3 USB_OTG, J4 IPEX RF Coaxial Connector SMD, M1 MODULE_RTL8188, U1 MT29F8G08ABABA, U2 ISL8022, U3 ALLWINNER-A13(176-LQFP), U4 TLV62569-SOT23-6, U5 TPS62233DRYR, U6 AS4C256M16D3A-12BAN(96-FBGA), U7 MCP130T-300ITT, Y1 Crystal_GND24_24MHz

Commit message: update Jan 8 2019
Connections:
- net PIN28 is gone; now on net PIN28_NDQS: GPIO1.27 (Pin_27)
- net PIN16_NCE0: now also RN2.1; no longer RN2.2
- net PIN18_NRB0: now also RN2.2; no longer RN2.1
Changed lines of the file:
@@
 $EndComp
 Wire Wire Line
-	2350 10800 3400 10800
-Wire Wire Line
-	3500 10950 3500 10800
-Wire Wire Line
-	2350 10950 3500 10950
+	2350 10950 3400 10950
 $Comp
 L Device:C_Small C28
@@
 Text Label 21550 8900 2    50   ~ 0
 PIN19_NRB1
-Text Label 19650 8900 0    50   ~ 0
-PIN28
 Text Label 21550 9000 2    50   ~ 0
 PIN29
@@
 Wire Wire Line
 	16650 12300 16650 12200
+$Comp
+L Mylib:+3.0VA #PWR0101
+U 1 1 5CE85E3A
+P 13150 8000
+F 0 "#PWR0101" H 13150 7850 50  0001 C CNN
+F 1 "+3.0VA" H 13165 8173 50  0000 C CNN
+F 2 "" H 13150 8000 50  0001 C CNN
+F 3 "" H 13150 8000 50  0001 C CNN
+	1    13150 8000
+	1    0    0    -1
+$EndComp
+Wire Wire Line
+	13150 8000 13150 8100
+Text Label 13150 8050 0    50   ~ 0
++3.0VA
+Wire Wire Line
+	2350 10800 3150 10800
+Wire Wire Line
+	3150 10850 3500 10850
+Wire Wire Line
+	3500 10850 3500 10800
+Wire Wire Line
+	3150 10800 3150 10850
+Wire Wire Line
+	3400 10950 3400 10800
 Wire Wire Line
 	2350 11250 3600 11250
@@
 Wire Bus Line
 	10950 1250 10950 6250
-$Comp
-L Mylib:+3.0VA #PWR0101
-U 1 1 5CE85E3A
-P 13150 8000
-F 0 "#PWR0101" H 13150 7850 50  0001 C CNN
-F 1 "+3.0VA" H 13165 8173 50  0000 C CNN
-F 2 "" H 13150 8000 50  0001 C CNN
-F 3 "" H 13150 8000 50  0001 C CNN
-	1    13150 8000
-	1    0    0    -1
-$EndComp
-Wire Wire Line
-	13150 8000 13150 8100
-Text Label 13150 8050 0    50   ~ 0
-+3.0VA
+Text Label 19650 8900 0    50   ~ 0
+PIN28_NDQS
 $EndSCHEMATC

Commit message: update March 52019
Parts:
- DEBUG1: footprint Connector_PinHeader_2.54mm:PinHeader_1x03_P2.54mm_Horizontal -> Connector_Molex:Molex_CLIK-Mate_502585-0370_1x03-1MP_P1.50mm_Horizontal
Connections:
- net REST-N is gone; now on net RESET-N: GPIO1.5 (Pin_5)
Changed lines of the file:
@@
 F 0 "DEBUG1" H 20480 2892 50  0000 L CNN
 F 1 "Conn_01x03" H 20480 2801 50  0000 L CNN
-F 2 "Connector_PinHeader_2.54mm:PinHeader_1x03_P2.54mm_Horizontal" H 20400 2850 50  0001 C CNN
+F 2 "Connector_Molex:Molex_CLIK-Mate_502585-0370_1x03-1MP_P1.50mm_Horizontal" H 20400 2850 50  0001 C CNN
 F 3 "~" H 20400 2850 50  0001 C CNN
 	1    20400 2850
@@
 	20850 9600 21550 9600
 Text Label 19650 7800 0    50   ~ 0
-REST-N
+RESET-N
 Text Label 19650 11200 0    50   ~ 0
 PIN4_TWI0-SCK
@@
 Wire Wire Line
 	3400 10950 3400 10800
+Text Label 19650 8900 0    50   ~ 0
+PIN28_NDQS
 Wire Wire Line
 	2350 11250 3600 11250
@@
 Wire Bus Line
 	10950 1250 10950 6250
-Text Label 19650 8900 0    50   ~ 0
-PIN28_NDQS
 $EndSCHEMATC

Commit message: update March 6 2019
Connections:
- net LCD-CLK: now also GPIO1.27 (Pin_27); no longer GPIO1.63 (Pin_63)
- net LCD-D10: now also GPIO1.51 (Pin_51); no longer GPIO1.54 (Pin_54)
- net LCD-D11: now also GPIO1.49 (Pin_49); no longer GPIO1.53 (Pin_53)
- net LCD-D12: now also GPIO1.47 (Pin_47); no longer GPIO1.52 (Pin_52)
- net LCD-D13: now also GPIO1.45 (Pin_45); no longer GPIO1.51 (Pin_51)
- net LCD-D14: now also GPIO1.43 (Pin_43); no longer GPIO1.50 (Pin_50)
- net LCD-D15: now also GPIO1.41 (Pin_41); no longer GPIO1.49 (Pin_49)
- net LCD-D18: now also GPIO1.39 (Pin_39); no longer GPIO1.48 (Pin_48)
- net LCD-D19: now also GPIO1.37 (Pin_37); no longer GPIO1.47 (Pin_47)
- net LCD-D2: now also GPIO1.63 (Pin_63); no longer GPIO1.59 (Pin_59)
- net LCD-D20: now also GPIO1.35 (Pin_35); no longer GPIO1.46 (Pin_46)
- net LCD-D21: now also GPIO1.33 (Pin_33); no longer GPIO1.45 (Pin_45)
- net LCD-D22: now also GPIO1.31 (Pin_31); no longer GPIO1.44 (Pin_44)
- net LCD-D23: now also GPIO1.29 (Pin_29); no longer GPIO1.43 (Pin_43)
- net LCD-D3: now also GPIO1.61 (Pin_61); no longer GPIO1.60 (Pin_60)
- net LCD-D4: now also GPIO1.59 (Pin_59); no longer GPIO1.57 (Pin_57)
- net LCD-D5: now also GPIO1.57 (Pin_57); no longer GPIO1.58 (Pin_58)
- net LCD-D7: now also GPIO1.53 (Pin_53); no longer GPIO1.56 (Pin_56)
- net LCD-DE: now also GPIO1.25 (Pin_25); no longer GPIO1.64 (Pin_64)
- net LCD-HSYNC: now also GPIO1.23 (Pin_23); no longer GPIO1.61 (Pin_61)
- net LCD-VSYNC: now also GPIO1.21 (Pin_21); no longer GPIO1.62 (Pin_62)
- net PIN10_TWI1-SCK: now also GPIO1.56 (Pin_56); no longer GPIO1.37 (Pin_37)
- net PIN11_TWI1-SDA: now also GPIO1.54 (Pin_54); no longer GPIO1.35 (Pin_35)
- net PIN15_NCE1: now also GPIO1.52 (Pin_52); no longer GPIO1.13 (Pin_13)
- net PIN19_NRB1: now also GPIO1.50 (Pin_50); no longer GPIO1.28 (Pin_28)
- net PIN28_NDQS: now also GPIO1.48 (Pin_48); no longer GPIO1.27 (Pin_27)
- net PIN29: now also GPIO1.46 (Pin_46); no longer GPIO1.30 (Pin_30)
- net PIN30: now also GPIO1.44 (Pin_44); no longer GPIO1.29 (Pin_29)
- net PIN31: now also GPIO1.42 (Pin_42); no longer GPIO1.26 (Pin_26)
- net PIN32: now also GPIO1.40 (Pin_40); no longer GPIO1.25 (Pin_25)
- net PIN33: now also GPIO1.38 (Pin_38); no longer GPIO1.24 (Pin_24)
- net PIN34: now also GPIO1.36 (Pin_36); no longer GPIO1.23 (Pin_23)
- net PIN35: now also GPIO1.34 (Pin_34); no longer GPIO1.22 (Pin_22)
- net PIN36: now also GPIO1.32 (Pin_32); no longer GPIO1.21 (Pin_21)
- net PIN37_LED1: now also GPIO1.30 (Pin_30); no longer GPIO1.12 (Pin_12)
- net PIN38_VGA-DIS: now also GPIO1.28 (Pin_28); no longer GPIO1.11 (Pin_11)
- net PIN39_USBH-EN: now also GPIO1.26 (Pin_26); no longer GPIO1.10 (Pin_10)
- net PIN6_PWM0: now also GPIO1.64 (Pin_64); no longer GPIO1.41 (Pin_41)
- net PIN7: now also GPIO1.62 (Pin_62); no longer GPIO1.42 (Pin_42)
- net PIN8: now also GPIO1.60 (Pin_60); no longer GPIO1.39 (Pin_39)
- net PIN9: now also GPIO1.58 (Pin_58); no longer GPIO1.40 (Pin_40)
- net SPI2-CLK: now also GPIO1.16 (Pin_16); no longer GPIO1.33 (Pin_33)
- net SPI2-CS0: now also GPIO1.14 (Pin_14); no longer GPIO1.34 (Pin_34)
- net SPI2-MISO: now also GPIO1.15 (Pin_15); no longer GPIO1.31 (Pin_31)
- net SPI2-MOSI: now also GPIO1.13 (Pin_13); no longer GPIO1.32 (Pin_32)
- net TWI2-SCK: now also GPIO1.10 (Pin_10); no longer GPIO1.36 (Pin_36)
- net TWI2-SDA: now also GPIO1.12 (Pin_12); no longer GPIO1.38 (Pin_38)
- net USB0-DRV: now also GPIO1.24 (Pin_24); no longer GPIO1.14 (Pin_14)
- net USB0-IDDET: now also GPIO1.11 (Pin_11); no longer GPIO1.16 (Pin_16)
- net USB0-VBUSDET: now also GPIO1.22 (Pin_22); no longer GPIO1.15 (Pin_15)
Changed lines of the file:
@@
 Text Label 21550 11200 2    50   ~ 0
 PIN5_TWI0-SDA
-Text Label 19650 9600 0    50   ~ 0
+Text Label 21550 10700 2    50   ~ 0
 PIN6_PWM0
+Text Label 21550 10600 2    50   ~ 0
+PIN7
+Text Label 21550 10500 2    50   ~ 0
+PIN8
+Text Label 21550 10400 2    50   ~ 0
+PIN9
+Text Label 21550 10300 2    50   ~ 0
+PIN10_TWI1-SCK
+Text Label 21550 10200 2    50   ~ 0
+PIN11_TWI1-SDA
+Text Label 21550 10100 2    50   ~ 0
+PIN15_NCE1
+Text Label 21550 10000 2    50   ~ 0
+PIN19_NRB1
+Text Label 21550 9800 2    50   ~ 0
+PIN29
+Text Label 21550 9700 2    50   ~ 0
+PIN30
 Text Label 21550 9600 2    50   ~ 0
-PIN7
-Text Label 19650 9500 0    50   ~ 0
-PIN8
+PIN31
 Text Label 21550 9500 2    50   ~ 0
-PIN9
-Text Label 19650 9400 0    50   ~ 0
-PIN10_TWI1-SCK
-Text Label 19650 9300 0    50   ~ 0
-PIN11_TWI1-SDA
-Text Label 19650 8200 0    50   ~ 0
-PIN15_NCE1
+PIN32
+Text Label 21550 9400 2    50   ~ 0
+PIN33
+Text Label 21550 9300 2    50   ~ 0
+PIN34
+Text Label 21550 9200 2    50   ~ 0
+PIN35
+Text Label 21550 9000 2    50   ~ 0
+PIN37_LED1
 Text Label 21550 8900 2    50   ~ 0
-PIN19_NRB1
-Text Label 21550 9000 2    50   ~ 0
-PIN29
-Text Label 19650 9000 0    50   ~ 0
-PIN30
+PIN38_VGA-DIS
 Text Label 21550 8800 2    50   ~ 0
-PIN31
-Text Label 19650 8800 0    50   ~ 0
-PIN32
-Text Label 21550 8700 2    50   ~ 0
-PIN33
-Text Label 19650 8700 0    50   ~ 0
-PIN34
-Text Label 21550 8600 2    50   ~ 0
-PIN35
-Text Label 21550 8100 2    50   ~ 0
-PIN37_LED1
-Text Label 19650 8100 0    50   ~ 0
-PIN38_VGA-DIS
-Text Label 21550 8000 2    50   ~ 0
 PIN39_USBH-EN
 Text Label 21550 7900 2    50   ~ 0
@@
 Wire Wire Line
 	12900 12300 13850 12300
-Text Label 21550 9900 2    50   ~ 0
+Text Label 19650 9500 0    50   ~ 0
 LCD-D18
-Text Label 21550 9800 2    50   ~ 0
+Text Label 19650 9300 0    50   ~ 0
 LCD-D20
-Text Label 21550 9700 2    50   ~ 0
+Text Label 19650 9100 0    50   ~ 0
 LCD-D22
-Text Label 21550 10200 2    50   ~ 0
+Text Label 19650 10100 0    50   ~ 0
 LCD-D10
-Text Label 21550 10100 2    50   ~ 0
+Text Label 19650 9900 0    50   ~ 0
 LCD-D12
-Text Label 21550 10000 2    50   ~ 0
+Text Label 19650 9700 0    50   ~ 0
 LCD-D14
+Text Label 19650 10700 0    50   ~ 0
+LCD-D2
 Text Label 19650 10500 0    50   ~ 0
-LCD-D2
-Text Label 19650 10400 0    50   ~ 0
 LCD-D4
 Text Label 19650 10300 0    50   ~ 0
 LCD-D6
-Text Label 19650 10600 0    50   ~ 0
+Text Label 19650 8700 0    50   ~ 0
 LCD-HSYNC
-Text Label 19650 10700 0    50   ~ 0
+Text Label 19650 8900 0    50   ~ 0
 LCD-CLK
 Text Label 19650 10800 0    50   ~ 0
@@
 Text Label 21550 10800 2    50   ~ 0
 TPX2
-Text Label 21550 10700 2    50   ~ 0
+Text Label 19650 8800 0    50   ~ 0
 LCD-DE
-Text Label 21550 10600 2    50   ~ 0
+Text Label 19650 8600 0    50   ~ 0
 LCD-VSYNC
-Text Label 21550 10300 2    50   ~ 0
+Text Label 19650 10200 0    50   ~ 0
 LCD-D7
-Text Label 21550 10400 2    50   ~ 0
+Text Label 19650 10400 0    50   ~ 0
 LCD-D5
-Text Label 21550 10500 2    50   ~ 0
+Text Label 19650 10600 0    50   ~ 0
 LCD-D3
+Text Label 19650 9600 0    50   ~ 0
+LCD-D15
+Text Label 19650 9800 0    50   ~ 0
+LCD-D13
 Text Label 19650 10000 0    50   ~ 0
-LCD-D15
-Text Label 19650 10100 0    50   ~ 0
-LCD-D13
-Text Label 19650 10200 0    50   ~ 0
 LCD-D11
-Text Label 19650 9700 0    50   ~ 0
+Text Label 19650 9000 0    50   ~ 0
 LCD-D23
-Text Label 19650 9800 0    50   ~ 0
+Text Label 19650 9200 0    50   ~ 0
 LCD-D21
-Text Label 19650 9900 0    50   ~ 0
+Text Label 19650 9400 0    50   ~ 0
 LCD-D19
 Text Label 21550 8400 2    50   ~ 0
@@
 Text Label 19650 8000 0    50   ~ 0
 LRADC
-Text Label 21550 9200 2    50   ~ 0
+Text Label 21550 8200 2    50   ~ 0
 SPI2-CS0
-Text Label 19650 9200 0    50   ~ 0
+Text Label 21550 8300 2    50   ~ 0
 SPI2-CLK
-Text Label 21550 9100 2    50   ~ 0
+Text Label 19650 8200 0    50   ~ 0
 SPI2-MOSI
-Text Label 19650 9100 0    50   ~ 0
+Text Label 19650 8300 0    50   ~ 0
 SPI2-MISO
 Text Label 19650 7900 0    50   ~ 0
 UBOOT
-Text Label 21550 9400 2    50   ~ 0
+Text Label 21550 8100 2    50   ~ 0
 TWI2-SDA
-Text Label 21550 9300 2    50   ~ 0
+Text Label 21550 8000 2    50   ~ 0
 TWI2-SCK
-Text Label 21550 8200 2    50   ~ 0
+Text Label 21550 8700 2    50   ~ 0
 USB0-DRV
-Text Label 21550 8300 2    50   ~ 0
+Text Label 19650 8100 0    50   ~ 0
 USB0-IDDET
-Text Label 19650 8300 0    50   ~ 0
+Text Label 21550 8600 2    50   ~ 0
 USB0-VBUSDET
 $Comp
@@
 Wire Wire Line
 	13150 9150 13900 9150
-Text Label 19650 8600 0    50   ~ 0
+Text Label 21550 9100 2    50   ~ 0
 PIN36
 Text Label 19650 11100 0    50   ~ 0
@@
 Wire Wire Line
 	3400 10950 3400 10800
-Text Label 19650 8900 0    50   ~ 0
+Text Label 21550 9900 2    50   ~ 0
 PIN28_NDQS
 Wire Wire Line

Commit message: finished VIGOLENO SBC PCB layout
Parts:
- Y1: symbol Device:Crystal_GND24_Small -> vigoleno-rescue:Crystal_GND24_Small-Device
- renumbered DEBUG1 to DEBUG, ENTER1 to ENTER, GPIO1 to GPIO, H-P1 to H-P, HOME1 to HOME, LED1 to LED, MENU1 to MENU, MIC1 to MIC, ON1 to ON, RESET1 to RESET, VOL+1 to VOL+, VOL-1 to VOL-
Connections:
- net +1.5V: now also C72.1, C74.1, C75.1, C76.1, C77.1, C78.1, C79.1, C81.1, C84.1, C85.1, C86.1, C88.1, C89.1, C91.1, C92.1, C93.1, C94.1, C96.1, U6.A1 (VDDQ), U6.A8 (VDDQ), U6.B2 (VDD), U6.C1 (VDDQ), U6.C9 (VDDQ), U6.D2 (VDDQ), U6.D9 (VDD), U6.E9 (VDDQ), U6.F1 (VDDQ), U6.G7 (VDD), U6.H2 (VDDQ), U6.H9 (VDDQ), U6.K2 (VDD), U6.K8 (VDD), U6.N1 (VDD), U6.N9 (VDD), U6.R1 (VDD), U6.R9 (VDD); no longer C42.1, C45.1, C51.1, C52.1, C54.1, U3.23 (VCC1_DRAM), U3.30 (VCC2_DRAM), U3.43 (VCC3_DRAM), U3.53 (VCC4_DRAM), U3.62 (VCC5_DRAM)
- new net: C42.1, C45.1, C51.1, C52.1, C54.1, U3.23 (VCC1_DRAM), U3.30 (VCC2_DRAM), U3.43 (VCC3_DRAM), U3.53 (VCC4_DRAM), U3.62 (VCC5_DRAM)
Changed lines of the file:
@@
 	1400 2850 4100 2850
 $Comp
-L Device:Crystal_GND24_Small Y1
+L vigoleno-rescue:Crystal_GND24_Small-Device Y1
 U 1 1 5BC34E7A
 P 4750 5000
@@
 Connection ~ 1400 6600
 $Comp
-L Mylib:APJ3-095S64 H-P1
+L Mylib:APJ3-095S64 H-P
 U 1 1 5BD47090
 P 1405 8035
-F 0 "H-P1" H 1400 8170 50  0000 C CNN
+F 0 "H-P" H 1400 8170 50  0000 C CNN
 F 1 "APJ3-095S64" H 1400 8070 50  0000 C CNN
 F 2 "MyKiCadLib:APJ3-095S64(Board_Cutout)" H 1300 8020 50  0001 C CNN
@@
 	2405 7550 3150 7550
 $Comp
-L Mylib:APJ3-095S64 MIC1
+L Mylib:APJ3-095S64 MIC
 U 1 1 5BD46FFE
 P 1405 7235
-F 0 "MIC1" H 1464 7395 50  0000 C CNN
+F 0 "MIC" H 1464 7395 50  0000 C CNN
 F 1 "APJ3-095S64" H 1464 7304 50  0000 C CNN
 F 2 "MyKiCadLib:APJ3-095S64(Board_Cutout)" H 1300 7220 50  0001 C CNN
@@
 	12800 12300 12900 12400
 $Comp
-L Mylib:4PIN_3.5x4.7_SMD VOL+1
+L Mylib:4PIN_3.5x4.7_SMD VOL+
 U 1 1 5BFB133A
 P 14100 8650
-F 0 "VOL+1" V 14079 8638 50  0000 L CNN
+F 0 "VOL+" V 14079 8638 50  0000 L CNN
 F 1 "4PIN_3.5x4.7_SMD" V 14170 8638 50  0000 L CNN
 F 2 "MyKiCadLib:4PIN_3.5x4.7_SMD" H 14100 8650 50  0001 C CNN
@@
 $EndComp
 $Comp
-L Mylib:4PIN_3.5x4.7_SMD VOL-1
+L Mylib:4PIN_3.5x4.7_SMD VOL-
 U 1 1 5BFB495B
 P 15000 8650
-F 0 "VOL-1" V 14979 8638 50  0000 L CNN
+F 0 "VOL-" V 14979 8638 50  0000 L CNN
 F 1 "4PIN_3.5x4.7_SMD" V 15070 8638 50  0000 L CNN
 F 2 "MyKiCadLib:4PIN_3.5x4.7_SMD" H 15000 8650 50  0001 C CNN
@@
 $EndComp
 $Comp
-L Mylib:4PIN_3.5x4.7_SMD MENU1
+L Mylib:4PIN_3.5x4.7_SMD MENU
 U 1 1 5BFB558B
 P 15900 8650
-F 0 "MENU1" V 15879 8638 50  0000 L CNN
+F 0 "MENU" V 15879 8638 50  0000 L CNN
 F 1 "4PIN_3.5x4.7_SMD" V 15970 8638 50  0000 L CNN
 F 2 "MyKiCadLib:4PIN_3.5x4.7_SMD" H 15900 8650 50  0001 C CNN
@@
 $EndComp
 $Comp
-L Mylib:4PIN_3.5x4.7_SMD ENTER1
+L Mylib:4PIN_3.5x4.7_SMD ENTER
 U 1 1 5BFB583C
 P 16800 8650
-F 0 "ENTER1" V 16779 8638 50  0000 L CNN
+F 0 "ENTER" V 16779 8638 50  0000 L CNN
 F 1 "4PIN_3.5x4.7_SMD" V 16870 8638 50  0000 L CNN
 F 2 "MyKiCadLib:4PIN_3.5x4.7_SMD" H 16800 8650 50  0001 C CNN
@@
 $EndComp
 $Comp
-L Mylib:4PIN_3.5x4.7_SMD HOME1
+L Mylib:4PIN_3.5x4.7_SMD HOME
 U 1 1 5BFB76F4
 P 17700 8650
-F 0 "HOME1" V 17679 8638 50  0000 L CNN
+F 0 "HOME" V 17679 8638 50  0000 L CNN
 F 1 "4PIN_3.5x4.7_SMD" V 17770 8638 50  0000 L CNN
 F 2 "MyKiCadLib:4PIN_3.5x4.7_SMD" H 17700 8650 50  0001 C CNN
@@
 $EndComp
 $Comp
-L Connector_Generic:Conn_01x03 DEBUG1
+L Connector_Generic:Conn_01x03 DEBUG
 U 1 1 5E8FB690
 P 20400 2850
-F 0 "DEBUG1" H 20480 2892 50  0000 L CNN
+F 0 "DEBUG" H 20480 2892 50  0000 L CNN
 F 1 "Conn_01x03" H 20480 2801 50  0000 L CNN
 F 2 "Connector_Molex:Molex_CLIK-Mate_502585-0370_1x03-1MP_P1.50mm_Horizontal" H 20400 2850 50  0001 C CNN
@@
 	10950 1250 12700 1250
 $Comp
-L Device:LED LED1
+L Device:LED LED
 U 1 1 5BF99DB8
 P 14200 9950
-F 0 "LED1" H 14192 9695 50  0000 C CNN
+F 0 "LED" H 14192 9695 50  0000 C CNN
 F 1 "LED0603" H 14192 9786 50  0000 C CNN
 F 2 "LED_SMD:LED_0603_1608Metric" H 14200 9950 50  0001 C CNN
@@
 	18800 6600 18800 850
 $Comp
-L Device:LED ON1
+L Device:LED ON
 U 1 1 6B858FB1
 P 16150 14900
-F 0 "ON1" V 16188 14783 50  0000 R CNN
+F 0 "ON" V 16188 14783 50  0000 R CNN
 F 1 "LED0603" V 16097 14783 50  0000 R CNN
 F 2 "LED_SMD:LED_0603_1608Metric" H 16150 14900 50  0001 C CNN
@@
 	5000 11350 5500 11350
 $Comp
-L Switch:SW_Push RESET1
+L Switch:SW_Push RESET
 U 1 1 5C1F72A0
 P 16350 10000
-F 0 "RESET1" H 16350 10285 50  0000 C CNN
+F 0 "RESET" H 16350 10285 50  0000 C CNN
 F 1 "SW_Push" H 16350 10194 50  0000 C CNN
 F 2 "MyKiCadLib:SW_3x6x5_2Pin_SMD" H 16350 10200 50  0001 C CNN
@@
 Text Label 4800 1250 0    50   ~ 0
 +1.2V-INT
-Text Label 5200 1250 0    50   ~ 0
+Text Label 17050 1350 0    50   ~ 0
 +1.5V
 Text Label 5450 1250 0    50   ~ 0
@@
 	13850 14100 13850 14250
 $Comp
-L Connector_Generic:Conn_02x40_Odd_Even GPIO1
+L Connector_Generic:Conn_02x40_Odd_Even GPIO
 U 1 1 5C17498A
 P 20550 9500
-F 0 "GPIO1" H 20600 11617 50  0000 C CNN
+F 0 "GPIO" H 20600 11617 50  0000 C CNN
 F 1 "Conn_02x40_Odd_Even" H 20600 11526 50  0000 C CNN
 F 2 "MyKiCadLib:2x40_pitch 0.8mm_SMD_header" H 20550 9500 50  0001 C CNN
